File: ImageProc.brd (EAGLE design)
At the start: 49.8 x 23.2 mm, 119 parts, among them IC1 XC61GC3002HR-G, IC10 AT45DB642D-CNU, IC2 MIC5335-SPYMT, IC3 MIC5335-JGYMT, IC4 DSPIC33FJ128MC706A, IC5 AT86RF233-ZU, IC6 LTC6088, IC7 DRV8833RTY, IC8 DRV8833RTY, IC9 MPU-6000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

Commit message: Initial replacement of dsPIC with STM32 chip in schematic.
Parts:
- removed IC4: DSPIC33FJ128MC706A, biomimetic:TQFP-64
- removed JP4: 51441-2493-C, biomimetic:MOLEX_52740-2490
- removed OSC1: ECS-2033-400, biomimetic:OSCILLATOR-SMD
- added IC11: STM32F405RGT, biomimetic:LQFP64
Connections:
- removed net 40MHZ: IC4.39, JP4.12, OSC1.3
- removed net CAM_D0: IC4.46, JP4.6
- removed net CAM_D1: IC4.49, JP4.4
- removed net CAM_D2: IC4.50, JP4.3
- removed net CAM_D3: IC4.51, JP4.5
- removed net CAM_D4: IC4.52, JP4.7
- removed net CAM_D5: IC4.53, JP4.9
- removed net CAM_D6: IC4.54, JP4.11
- removed net CAM_D7: IC4.55, JP4.13
- removed net CAM_PCLK: IC4.59, JP4.8
- removed net CAM_PWDN: IC4.48, JP4.17
- removed net CAM_VSYNC: IC4.47, JP4.18
- new net VBAT: IC11.1
- new net VDD: IC11.19, IC11.32, IC11.48, IC11.64
- new net VDDA: IC11.13
- new net VSS: IC11.18, IC11.63
- new net VSSA: IC11.12
- net !RESET: no longer IC4.7
- net !SS1: no longer IC4.14
- net !SS2_1: no longer IC4.8
- net !SS2_2: no longer IC4.40
- net 1.8V: no longer JP4.15
- net 2.5V: no longer JP4.14, JP4.21
- net 3.3V: no longer IC4.10, IC4.26, IC4.38, IC4.57, OSC1.4
- net AN1/RB1: no longer IC4.15
- net AN3/INDX/RB3: no longer IC4.13
- net AN4/QEA/IC7/RB4: no longer IC4.12
- net AN5/QEB/IC8/RB5: no longer IC4.11
- net BATT_LEVEL: no longer IC4.16
- net CAM_HREF: no longer IC4.58, JP4.16
- net GND: no longer IC4.20, IC4.25, IC4.41, IC4.9, JP4.10, JP4.19, JP4.23, OSC1.2
- net GN_LED: no longer IC4.28
- net IC3/INT3/RD10: no longer IC4.44
- net IMU_IRQ: no longer IC4.42
- net LOWBATT_IRQ: no longer IC4.43
- net MOTOR_A_BEMF: no longer IC4.21
- net MOTOR_A_IN1: no longer IC4.61
- net MOTOR_A_IN2: no longer IC4.60
- net MOTOR_B_BEMF: no longer IC4.22
- net MOTOR_B_IN1: no longer IC4.63
- net MOTOR_B_IN2: no longer IC4.62
- net MOTOR_C_BEMF: no longer IC4.23
- net MOTOR_C_IN1: no longer IC4.1
- net MOTOR_C_IN2: no longer IC4.64
- net MOTOR_D_BEMF: no longer IC4.24
- net MOTOR_D_IN1: no longer IC4.3
- net MOTOR_D_IN2: no longer IC4.2
- net N$21: no longer IC4.19
- net N$28: no longer IC4.56
- net PGC: no longer IC4.17
- net PGD: no longer IC4.18
- net RADIO_IRQ: no longer IC4.45
- net RADIO_SLP_TR: no longer IC4.30
- net RD_LED: no longer IC4.27
- net SCK1: no longer IC4.35
- net SCK2: no longer IC4.4
- net SCL1: no longer IC4.37, JP4.20
- net SDA1: no longer IC4.36, JP4.22
- net SDI1: no longer IC4.34
- net SDI2: no longer IC4.5
- net SDO1: no longer IC4.33
- net SDO2: no longer IC4.6
- net U2RX: no longer IC4.31
- net U2TX: no longer IC4.32
- net YW_LED: no longer IC4.29
Routing:
- net 40MHZ: track 38.6 -> 0.00 mm, vias 2 -> 0
- net SDA1: track 45.6 -> 13.0 mm, vias 4 -> 1
- net CAM_VSYNC: track 32.0 -> 0.00 mm, vias 1 -> 0
- net CAM_D0: track 31.9 -> 0.00 mm, vias 2 -> 0
- net CAM_D6: track 31.3 -> 0.00 mm, vias 2 -> 0
- net CAM_PWDN: track 31.2 -> 0.00 mm, vias 1 -> 0
- net CAM_D7: track 27.6 -> 0.00 mm, vias 2 -> 0
- net CAM_HREF: track 35.7 -> 8.46 mm, vias 3 -> 1
- net CAM_D1: track 26.6 -> 0.00 mm, vias 2 -> 0
- net CAM_D4: track 25.4 -> 0.00 mm, vias 2 -> 0
- net CAM_D2: track 25.3 -> 0.00 mm, vias 2 -> 0
- net CAM_PCLK: track 24.7 -> 0.00 mm, vias 2 -> 0
- net CAM_D5: track 22.7 -> 0.00 mm, vias 2 -> 0
- net CAM_D3: track 22.6 -> 0.00 mm, vias 2 -> 0
- net MOTOR_C_IN1: track 34.5 -> 24.5 mm, vias 2 -> 1
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